Commit message: fix elp gazebo xacro

File: andante_description/urdf/sensors/elp.gazebo.xacro (robot description, xacro)
@@ -3,5 +3,4 @@
     <xacro:macro name="elp_gazebo" params="prefix">
         <gazebo reference="${prefix}elp_camera_link">
-            <material>Gazebo/Green</material>
             <visualize>true</visualize>
             <turnGravityOff>false</turnGravityOff>
