Commit message: add azure_kinect urdf

File: andante_description/urdf/andante.urdf.xacro (robot description, xacro)
@@ -3,7 +3,11 @@
   <xacro:include filename="$(find andante_description)/urdf/base/andante_base.urdf.xacro" />
   <xacro:include filename="$(find andante_description)/urdf/sensors/ld06.urdf.xacro" />
+  <xacro:include filename="$(find andante_description)/urdf/sensors/azure_kinect.urdf.xacro" />
   <xacro:andante_base wheel_separation="0.235" base_diameter="0.3485" />
   <xacro:ld06 parent="base_link">
     <origin xyz="-0.0471 0 0.09595" rpy="0 0 ${PI}" />
   </xacro:ld06>
+  <xacro:azure_kinect parent="base_link">
+    <origin xyz="0 0 0.25" rpy="0 0 0" />
+  </xacro:azure_kinect>
 </robot>

Commit message: fix urdf

File: andante_description/urdf/andante.urdf.xacro (robot description, xacro)
@@ -1,13 +1,10 @@
-<?xml version="1.0" ?>
+<?xml version="1.0"?>
 <robot name="andante" xmlns:xacro="http://ros.org/wiki/xacro">
-  <xacro:include filename="$(find andante_description)/urdf/base/andante_base.urdf.xacro" />
-  <xacro:include filename="$(find andante_description)/urdf/sensors/ld06.urdf.xacro" />
-  <xacro:include filename="$(find andante_description)/urdf/sensors/azure_kinect.urdf.xacro" />
-  <xacro:andante_base wheel_separation="0.235" base_diameter="0.3485" />
-  <xacro:ld06 parent="base_link">
-    <origin xyz="-0.0471 0 0.09595" rpy="0 0 ${PI}" />
-  </xacro:ld06>
-  <xacro:azure_kinect parent="base_link">
-    <origin xyz="0 0 0.25" rpy="0 0 0" />
-  </xacro:azure_kinect>
+  <xacro:include filename="$(find create_description)/urdf/create_base.urdf.xacro" />
+  <xacro:include filename="$(find create_description)/urdf/create_2_gazebo.urdf.xacro" />
+  <xacro:create_base wheel_separation="0.235" base_diameter="0.3485">
+    <mesh filename="package://create_description/meshes/create_2.dae" />
+  </xacro:create_base>
 </robot>
+Name: YesNoButton
+Name: YesNoButton

Commit message: fix mesh path for gazebo
https://answers.ros.org/question/396756/gazebo-doesnt-find-mesh-file-in-urdf/

File: andante_description/urdf/andante.urdf.xacro (robot description, xacro)
@@ -2,7 +2,6 @@
 <robot name="andante" xmlns:xacro="http://ros.org/wiki/xacro">
   <xacro:include filename="$(find create_description)/urdf/create_base.urdf.xacro" />
-  <xacro:include filename="$(find create_description)/urdf/create_2_gazebo.urdf.xacro" />
   <xacro:create_base wheel_separation="0.235" base_diameter="0.3485">
-    <mesh filename="package://create_description/meshes/create_2.dae" />
+    <mesh filename="$(find create_description)/meshes/create_2.dae" />
   </xacro:create_base>
 </robot>

Commit message: update urdf

File: andante_description/urdf/andante.urdf.xacro (robot description, xacro)
@@ -3,5 +3,13 @@
   <xacro:include filename="$(find create_description)/urdf/create_base.urdf.xacro" />
   <xacro:create_base wheel_separation="0.235" base_diameter="0.3485">
-    <mesh filename="$(find create_description)/meshes/create_2.dae" />
+    <mesh filename="package://create_description/meshes/create_2.dae" />
   </xacro:create_base>
+  <xacro:include filename="$(find andante_description)/urdf/sensors/plate.urdf.xacro" />
+  <xacro:plate prefix="" parent="base_link">
+    <origin xyz="0 0 0.0713" rpy="0 0 0" />
+  </xacro:plate>
+  <xacro:include filename="$(find andante_description)/urdf/sensors/elp.urdf.xacro" />
+  <xacro:elp prefix="" parent="plate_link">
+    <origin xyz="0 0 0.065" rpy="0 0 0" />
+  </xacro:elp>
 </robot>

Commit message: Gazebo Simulatior (#11)
* create package

* add world of petitcon

* add elp.*.xacro

* add plate.urdf.xacro

* fix mesh path for gazebo

https://answers.ros.org/question/396756/gazebo-doesnt-find-mesh-file-in-urdf/

* fix elp xacro

* update urdf

* add spawn robot in petitcon launch

* patch create_robot for gazebo11+foxy

* update create_robot

* add collision to petitcon world

* fix plate urdf path

* fix elp camera urdf angle

* fix elp gazebo xacro

* fix spawn yaw angle

File: andante_description/urdf/andante.urdf.xacro (robot description, xacro)
@@ -2,7 +2,14 @@
 <robot name="andante" xmlns:xacro="http://ros.org/wiki/xacro">
   <xacro:include filename="$(find create_description)/urdf/create_base.urdf.xacro" />
-  <xacro:include filename="$(find create_description)/urdf/create_2_gazebo.urdf.xacro" />
   <xacro:create_base wheel_separation="0.235" base_diameter="0.3485">
     <mesh filename="package://create_description/meshes/create_2.dae" />
   </xacro:create_base>
+  <xacro:include filename="$(find andante_description)/urdf/plate.urdf.xacro" />
+  <xacro:plate prefix="" parent="base_link">
+    <origin xyz="0 0 0.0713" rpy="0 0 0" />
+  </xacro:plate>
+  <xacro:include filename="$(find andante_description)/urdf/sensors/elp.urdf.xacro" />
+  <xacro:elp prefix="" parent="plate_link">
+    <origin xyz="0 0 0.065" rpy="0 0 0" />
+  </xacro:elp>
 </robot>
